File: rfidAndPOE.sch (KiCad schematic (older format))
At the start: 51 parts, among them Q1 Si3440DV, NFET, Q2 MMBTA42, Q3 2N7002

Commit message: Created a symbol for the RJ45 connector and hooked it up to the PoE stuff. Placed enc28j60, but haven't connected anything to it. May have added an extra library to the project file on accident.
Parts:
- added J?: 0813-1X1T-57-F, symbol 0813-1X1T-57-F
- added U?: ENC28J60, symbol ENC28J60
Connections:
- net labels added: Ethernet+, Ethernet-, EthernetSpare+, EthernetSpare-
- wire segments 114 -> 122

Commit message: Added 5V to 3.3V buck converter.
Parts:
- added C? (x2): 10nF, symbol CAPACITOR
- added C?: 100nF, symbol CAPACITOR
- added C? (x3): 10uF, symbol CAPACITOR
- added D? (x2): LED, symbol LED
- added D?: 1N4148, symbol DIODE
- added D?: 1N5189, symbol DIODESCH
- added L?: choke, symbol INDUCTOR_SMALL
- added L?: 15uH, symbol INDUCTOR_SMALL
- added R? (x4): 49R9,1%, symbol RESISTOR
- added R? (x2): RESISTOR, symbol RESISTOR
- added R?: 31.2k, symbol RESISTOR
- added R?: 10k, symbol RESISTOR
- added U?: MCP16301, symbol MCP16301
Connections:
- net labels added: 3V3, EVDD, EVddPLL, EVddRx, EVddTx, VddOSC
- wire segments 122 -> 192
Other:
- moved on the sheet: C1, C12, C13, C14, C2, C3, C4, C5, C6, C7, C8, C9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

Commit message: Added some text comments and a box around the 3.3V supply.
Other:
- note added: "5V to 3.3V@600mA buck supply"
- note added: "5V@1.8A"
Changed lines of the file:
@@
 Wire Wire Line
 	14040 1450 14040 1490
+Wire Notes Line
+	13530 615  13530 2080
+Wire Notes Line
+	13530 2080 17460 2080
+Wire Notes Line
+	17460 2080 17460 615
+Wire Notes Line
+	17460 615  13530 615
+Text Notes 15085 1965 2    60   ~ 0
+5V to 3.3V@600mA buck supply
+Text Notes 12320 755  2    60   ~ 0
+5V@1.8A
 $EndSCHEMATC

Commit message: Added a test point and power good LED to the 3.3V rail.
Parts:
- added D?: 3V3 LED, symbol LED
- added P?: TST, symbol TST
- added R?: 2.8k, symbol RESISTOR
Connections:
- wire segments 192 -> 196

Commit message: Added 12V boost supply.
Parts:
- added C?: 47nF, symbol CAPACITOR
- added C?: 180nF, symbol CAPACITOR
- added C? (x2): 10uF, symbol CAPACITOR
- added C?: 22uF, symbol CAPACITOR
- added D?: MBRA340T3G, symbol DIODE
- added D?: 12V LED, symbol LED
- added L?: 10uH, symbol INDUCTOR_SMALL
- added P?: TST, symbol TST
- added R?: 1.4k, symbol RESISTOR
- added R?: 143k, symbol RESISTOR
- added R?: 16.2k, symbol RESISTOR
- added R?: 226k, symbol RESISTOR
- added R?: 10k, symbol RESISTOR
- added U?: TPS61175, symbol TPS61175
Connections:
- net labels added: 12V
- wire segments 196 -> 241

Commit message: Added text to 12V supply and added a note about the 12V supply current limitations. Also relabeled some of the test points.
Parts:
- P?: value TST -> +3V3
- P?: value TST -> +12V
Other:
- note added: "5V to 12V@750mA boost supply"
- note added: "Note:\n12V@750mA is 9W\n5V@1.8A is 9W"
- moved on the sheet: D?, L?, P?, U?

Commit message: Missed the feedback connection to the IC in the 12V supply.
Parts:
- gave numbers to parts that had none: 53
Connections:
- wire segments 241 -> 242

Commit message: Fixed some wires that weren't actually connected.
Connections:
- wire segments 242 -> 246
Other:
- moved on the sheet: P1, P2, P3, P4
Changed lines of the file:
@@
 L TST P4
 U 1 1 52A279E6
-P 11500 905
-F 0 "P4" H 11500 1205 40  0000 C CNN
-F 1 "+5V" H 11500 1155 30  0000 C CNN
-F 2 "" H 11500 905 60  0000 C CNN
-F 3 "" H 11500 905 60  0000 C CNN
-	1    11500 905
+P 11500 870
+F 0 "P4" H 11500 1170 40  0000 C CNN
+F 1 "+5V" H 11500 1120 30  0000 C CNN
+F 2 "" H 11500 870 60  0000 C CNN
+F 3 "" H 11500 870 60  0000 C CNN
+	1    11500 870
 	1    0    0    -1
 $EndComp
@@
 L TST P3
 U 1 1 52A279FA
-P 11085 4515
-F 0 "P3" H 11085 4815 40  0000 C CNN
-F 1 "GND" H 11085 4765 30  0000 C CNN
-F 2 "" H 11085 4515 60  0000 C CNN
-F 3 "" H 11085 4515 60  0000 C CNN
-	1    11085 4515
+P 11085 4485
+F 0 "P3" H 11085 4785 40  0000 C CNN
+F 1 "GND" H 11085 4735 30  0000 C CNN
+F 2 "" H 11085 4485 60  0000 C CNN
+F 3 "" H 11085 4485 60  0000 C CNN
+	1    11085 4485
 	1    0    0    -1
 $EndComp
@@
 L TST P2
 U 1 1 52A27A0E
-P 2200 2260
-F 0 "P2" H 2200 2560 40  0000 C CNN
-F 1 "PoE+" H 2200 2510 30  0000 C CNN
-F 2 "" H 2200 2260 60  0000 C CNN
-F 3 "" H 2200 2260 60  0000 C CNN
-	1    2200 2260
+P 2200 2230
+F 0 "P2" H 2200 2530 40  0000 C CNN
+F 1 "PoE+" H 2200 2480 30  0000 C CNN
+F 2 "" H 2200 2230 60  0000 C CNN
+F 3 "" H 2200 2230 60  0000 C CNN
+	1    2200 2230
 	1    0    0    -1
 $EndComp
@@
 L TST P1
 U 1 1 52A27A22
-P 2145 3010
-F 0 "P1" H 2145 3310 40  0000 C CNN
-F 1 "PoE-" H 2145 3260 30  0000 C CNN
-F 2 "" H 2145 3010 60  0000 C CNN
-F 3 "" H 2145 3010 60  0000 C CNN
-	1    2145 3010
+P 2120 2995
+F 0 "P1" H 2120 3295 40  0000 C CNN
+F 1 "PoE-" H 2120 3245 30  0000 C CNN
+F 2 "" H 2120 2995 60  0000 C CNN
+F 3 "" H 2120 2995 60  0000 C CNN
+	1    2120 2995
 	1    0    0    -1
 $EndComp
@@
 Connection ~ 8710 4515
 Wire Wire Line
-	9630 4515 11575 4515
+	9625 4515 11575 4515
 Connection ~ 11575 1135
 Connection ~ 11575 1390
@@
 	16200 2745 17130 2745
 Wire Wire Line
-	16505 2885 16505 2745
+	16505 2745 16505 2890
 Connection ~ 16505 2745
 Wire Wire Line
@@
 	15535 3345 16505 3345
 Connection ~ 16505 3345
+Wire Wire Line
+	2120 2995 2120 3015
+Connection ~ 2120 3015
+Wire Wire Line
+	2200 2265 2200 2230
+Connection ~ 2200 2265
+Wire Wire Line
+	11085 4515 11085 4485
+Connection ~ 11085 4515
+Wire Wire Line
+	11500 870  11500 905
+Connection ~ 11500 905
 $EndSCHEMATC
