File: hardware/rfidAndPOE.kicad_pcb (KiCad board)
At the start: 4 copper layers, 100 x 50 mm, 127 parts, among them J1 0813-1X1T-57-F, J2 SWD, J3 MCU Port B, J4 MCU Port C, P1 PoE-, P2 PoE+, P3 GND, P4 +5V, P5 +12V, P6 +3V3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

Commit message: Added white rectangle for making notes on pcb
Routing:
- net (no net): track 0.00 -> 1.49 mm, vias 0 -> 3
- net GNDA: track 65.8 -> 64.3 mm, vias 17 -> 14
