File: hardware/POE.kicad_pcb (KiCad board)
At the start: 4 copper layers, 100 x 50 mm, 127 parts, among them J1 0813-1X1T-57-F, J2 SWD, J3 MCU Port B, J4 MCU Port C, P1 PoE-, P2 PoE+, P3 GND, P4 +5V, P5 +12V, P6 +3V3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

Commit message: Changed C5 to connect it to GNDA instead of VPortN. See http://jonneal.me/error-in-linear-tech-design-note-361/ for reason why.
Connections:
- C5 pad 2: Net-(C1-Pad2) -> GNDA
Routing:
- net Net-(C1-Pad2): track 33.0 -> 29.0 mm
- net GNDA: track 64.3 -> 68.3 mm
