File: hardware/POE/POE.sch (KiCad schematic (older format))
At the start: 122 parts, among them J1 0813-1X1T-57-F, J2 SWD, J3 MCU Port B, J4 MCU Port C, P1 PoE-, P2 PoE+, P3 GND, P4 +5V, P5 +12V, P6 +3V3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

Commit message: Reorganizing hardware folder in to separate folders for separate boards.
Parts:
- C1, C12, C13, C14, C15, C2, C3, C4, C6, C7, C8: symbol C -> C-RESCUE-POE
- C5, C9: symbol CP1 -> CP1-RESCUE-POE
- D10, D11, D12, D16, D17: symbol LED -> LED-RESCUE-POE
- R1, R10, R11, R12, R13, R14, R2, R21, R22, R3, R35, R36, R4, R400, R5, R6, R7, R8, R9: symbol R -> R-RESCUE-POE
