File: hardware/POEstamp/POE.sch (KiCad schematic (older format))
At the start: 57 parts, among them J1 0813-1X1T-57-F, P3 GND, P4 +5V, P5 CONN_01X05, P6 5Vout, P7 GNDout, Q1 SI3440DV, NFET, Q2 2N7002, Q3 MMBTA42, T1 PA1134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

Commit message: Fixed backwards LED and finished putting all components within the board outline. Everything should be close to its final location, all silk screens are aligned pretty alright.
Parts:
- removed D12: 5V LED, LEDs:LED-0603, symbol LED-RESCUE-POE
- added D12: 5V LED, LEDs:LED-0603, symbol LED
Connections:
- net GND: now also D12.1 (K)
- net at R22.2: now also D12.2 (A)
Changed lines of the file:
@@
 GNDA is the input ground from ethernet.\nGND is isolated ground.
-$Comp
-L LED-RESCUE-POE D12
-U 1 1 52A27A6E
-P 15270 3555
-F 0 "D12" H 15270 3655 50  0000 C CNN
-F 1 "5V LED" H 15275 3440 50  0000 C CNN
-F 2 "LEDs:LED-0603" H 15270 3555 60  0001 C CNN
-F 3 "http://www.osram-os.com/Graphics/XPic9/00128783_0.pdf" H 15270 3555 60  0001 C CNN
-F 4 "Digikey" H 15270 3555 60  0001 C CNN "Vend1"
-F 5 "475-1409-1-ND" H 15270 3555 60  0001 C CNN "Vend1Id"
-	1    15270 3555
-	0    1    1    0
-$EndComp
 $Comp
 L GND-RESCUE-POE #PWR013
@@
 Text Notes 6350 1800 0    59   ~ 0
 Several of the components in this area need thermal \nanalysis and replacement with appropriate packages.
+$Comp
+L LED D12
+U 1 1 5656CBC8
+P 15270 3555
+F 0 "D12" H 15270 3655 50  0000 C CNN
+F 1 "5V LED" H 15270 3455 50  0000 C CNN
+F 2 "LEDs:LED-0603" H 15270 3555 60  0001 C CNN
+F 3 "http://www.osram-os.com/Graphics/XPic9/00128783_0.pdf" H 15270 3555 60  0001 C CNN
+F 4 "Digikey" H 15270 3555 60  0001 C CNN "Vend1"
+F 5 "475-1409-1-ND" H 15270 3555 60  0001 C CNN "Vend1Id"
+	1    15270 3555
+	0    -1   -1   0
+$EndComp
 $EndSCHEMATC
